File: spi-port-expander/spi-port-expander.kicad_sch (KiCad schematic)
At the start: 12 parts, among them J1 Conn_01x14_Pin, J2 Conn_02x08_Top_Bottom, J3 Conn_02x01, U1 MCP23S17_SP

Commit message: Finish SPI port expander layout
Parts:
- removed J2: Conn_02x08_Top_Bottom, Connector_PinHeader_2.54mm:PinHeader_2x08_P2.54mm_Vertical, symbol Connector_Generic:Conn_02x08_Top_Bottom
- added J4: Conn_02x08_Odd_Even, Connector_PinHeader_2.54mm:PinHeader_2x08_P2.54mm_Vertical, symbol Connector_Generic:Conn_02x08_Odd_Even
- JP1, JP2, JP3: footprint Jumper:SolderJumper-3_P1.3mm_Open_RoundedPad1.0x1.5mm -> Jumper:SolderJumper-3_P1.3mm_Open_Pad1.0x1.5mm
Connections:
- net +3.3V: no longer C1.2
- net G0: now also J4.1 (Pin_1)
- net G1: now also J4.3 (Pin_3)
- net G10: now also J4.6 (Pin_6)
- net G11: now also J4.8 (Pin_8)
- net G12: now also J4.10 (Pin_10)
- net G13: now also J4.12 (Pin_12)
- net G14: now also J4.14 (Pin_14)
- net G15: now also J4.16 (Pin_16)
- net G2: now also J4.5 (Pin_5)
- net G3: now also J4.7 (Pin_7)
- net G4: now also J4.9 (Pin_9)
- net G5: now also J4.11 (Pin_11)
- net G6: now also J4.13 (Pin_13)
- net G7: now also J4.15 (Pin_15)
- net G8: now also J4.2 (Pin_2)
- net G9: now also J4.4 (Pin_4)
- net GND: now also C1.2
Changed lines of the file:
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@@
   (junction (at 160.02 74.93) (diameter 0) (color 0 0 0 0)
   )
-  (junction (at 53.34 43.18) (diameter 0) (color 0 0 0 0)
-  )
   (junction (at 101.6 62.23) (diameter 0) (color 0 0 0 0)
   )
@@
     (stroke (width 0) (type default))
   )
-  (wire (pts (xy 60.96 43.18) (xy 53.34 43.18))
-    (stroke (width 0) (type default))
-  )
   (wire (pts (xy 144.78 78.74) (xy 144.78 74.93))
     (stroke (width 0) (type default))
   )
-  (wire (pts (xy 53.34 33.02) (xy 53.34 43.18))
+  (wire (pts (xy 53.34 33.02) (xy 53.34 46.99))
     (stroke (width 0) (type default))
   )
@@
   )
   (wire (pts (xy 60.96 41.91) (xy 60.96 43.18))
-    (stroke (width 0) (type default))
-  )
-  (wire (pts (xy 53.34 43.18) (xy 53.34 46.99))
     (stroke (width 0) (type default))
   )
@@
   )
   (symbol (lib_id "Interface_Expansion:MCP23S17_SP") (at 53.34 74.93 0) (unit 1)
-    (in_bom yes) (on_board yes) (dnp no) (fields_autoplaced)
-    (property "Reference" "U1" (at 55.5341 46.99 0)
-      (effects (font (size 1.27 1.27)) (justify left))
-    )
-    (property "Value" "MCP23S17_SP" (at 55.5341 49.53 0)
+    (in_bom yes) (on_board yes) (dnp no)
+    (property "Reference" "U1" (at 43.18 45.72 0)
+      (effects (font (size 1.27 1.27)) (justify left))
+    )
+    (property "Value" "MCP23S17_SP" (at 36.83 48.26 0)
       (effects (font (size 1.27 1.27)) (justify left))
     )
@@
       (effects (font (size 1.27 1.27)) (justify left) hide)
     )
-    (property "Footprint" "Jumper:SolderJumper-3_P1.3mm_Open_RoundedPad1.0x1.5mm" (at 144.78 83.82 0)
+    (property "Footprint" "Jumper:SolderJumper-3_P1.3mm_Open_Pad1.0x1.5mm" (at 144.78 83.82 0)
       (effects (font (size 1.27 1.27)) hide)
     )
@@
         (path "/85439cc6-089f-4138-8a5b-34b6e0a5a6a8"
           (reference "JP1") (unit 1)
+        )
+      )
+    )
+  )
+  (symbol (lib_id "Connector_Generic:Conn_02x08_Odd_Even") (at 157.48 31.75 0) (unit 1)
+    (in_bom yes) (on_board yes) (dnp no) (fields_autoplaced)
+    (property "Reference" "J4" (at 158.75 17.78 0)
+      (effects (font (size 1.27 1.27)))
+    )
+    (property "Value" "Conn_02x08_Odd_Even" (at 158.75 20.32 0)
+      (effects (font (size 1.27 1.27)) hide)
+    )
+    (property "Footprint" "Connector_PinHeader_2.54mm:PinHeader_2x08_P2.54mm_Vertical" (at 157.48 31.75 0)
+      (effects (font (size 1.27 1.27)) hide)
+    )
+    (property "Datasheet" "~" (at 157.48 31.75 0)
+      (effects (font (size 1.27 1.27)) hide)
+    )
+    (pin "9")
+    (pin "16")
+    (pin "2")
+    (pin "12")
+    (pin "15")
+    (pin "14")
+    (pin "13")
+    (pin "10")
+    (pin "7")
+    (pin "8")
+    (pin "5")
+    (pin "4")
+    (pin "11")
+    (pin "1")
+    (pin "6")
+    (pin "3")
+    (instances
+      (project "spi-port-expander"
+        (path "/85439cc6-089f-4138-8a5b-34b6e0a5a6a8"
+          (reference "J4") (unit 1)
         )
       )
@@
       (effects (font (size 1.27 1.27)) (justify left) hide)
     )
-    (property "Footprint" "Jumper:SolderJumper-3_P1.3mm_Open_RoundedPad1.0x1.5mm" (at 160.02 83.82 0)
+    (property "Footprint" "Jumper:SolderJumper-3_P1.3mm_Open_Pad1.0x1.5mm" (at 160.02 83.82 0)
       (effects (font (size 1.27 1.27)) hide)
     )
@@
     )
   )
-  (symbol (lib_id "Connector_Generic:Conn_02x08_Top_Bottom") (at 157.48 31.75 0) (unit 1)
-    (in_bom yes) (on_board yes) (dnp no)
-    (property "Reference" "J2" (at 158.75 20.32 0)
-      (effects (font (size 1.27 1.27)))
-    )
-    (property "Value" "Conn_02x08_Top_Bottom" (at 158.75 20.32 0)
-      (effects (font (size 1.27 1.27)) hide)
-    )
-    (property "Footprint" "Connector_PinHeader_2.54mm:PinHeader_2x08_P2.54mm_Vertical" (at 157.48 31.75 0)
-      (effects (font (size 1.27 1.27)) hide)
-    )
-    (property "Datasheet" "~" (at 157.48 31.75 0)
-      (effects (font (size 1.27 1.27)) hide)
-    )
-    (pin "8")
-    (pin "15")
-    (pin "4")
-    (pin "6")
-    (pin "1")
-    (pin "2")
-    (pin "12")
-    (pin "14")
-    (pin "13")
-    (pin "11")
-    (pin "10")
-    (pin "7")
-    (pin "3")
-    (pin "9")
-    (pin "5")
-    (pin "16")
-    (instances
-      (project "spi-port-expander"
-        (path "/85439cc6-089f-4138-8a5b-34b6e0a5a6a8"
-          (reference "J2") (unit 1)
-        )
-      )
-    )
-  )
   (symbol (lib_id "Connector_Generic:Conn_02x01") (at 157.48 49.53 0) (unit 1)
     (in_bom yes) (on_board yes) (dnp no)
@@
       (effects (font (size 1.27 1.27)) (justify left) hide)
     )
-    (property "Footprint" "Jumper:SolderJumper-3_P1.3mm_Open_RoundedPad1.0x1.5mm" (at 175.26 83.82 0)
+    (property "Footprint" "Jumper:SolderJumper-3_P1.3mm_Open_Pad1.0x1.5mm" (at 175.26 83.82 0)
       (effects (font (size 1.27 1.27)) hide)
     )
@@
         )
       )
+    )
+  )
+  (symbol (lib_id "power:GND") (at 60.96 43.18 0) (unit 1)
+    (in_bom yes) (on_board yes) (dnp no) (fields_autoplaced)
+    (property "Reference" "#PWR08" (at 60.96 49.53 0)
+      (effects (font (size 1.27 1.27)) hide)
+    )
+    (property "Value" "GND" (at 60.96 48.26 0)
+      (effects (font (size 1.27 1.27)))
+    )
+    (property "Footprint" "" (at 60.96 43.18 0)
+      (effects (font (size 1.27 1.27)) hide)
+    )
+    (property "Datasheet" "" (at 60.96 43.18 0)
+      (effects (font (size 1.27 1.27)) hide)
+    )
+    (pin "1")
+    (instances
+      (project "spi-port-expander"
+        (path "/85439cc6-089f-4138-8a5b-34b6e0a5a6a8"
+          (reference "#PWR08") (unit 1)
+        )
+      )
