File: pwm-dc-dimmer/channel1.kicad_sch (KiCad schematic)
At the start: 2 parts, among them Q2 NMOS

Commit message: Add power routing
Parts:
- removed Q2: NMOS, symbol Simulation_SPICE:NMOS
- added D1: LED, LED_SMD:LED_0805_2012Metric, symbol Device:LED
- added Q1: Q_NMOS_GDS, Package_TO_SOT_SMD:TO-252-2, symbol Transistor_FET:Q_NMOS_GDS
- added R14, R26: 10K, Resistor_SMD:R_0805_2012Metric, symbol Device:R
- R3: footprint (none) -> Resistor_SMD:R_1206_3216Metric
Connections:
- net GATE_SINK: now also Q1.1 (G)
- net GND_LOAD: now also Q1.3 (S)
- net LOAD_ANODE: now also D1.1 (K), Q1.2 (D)
- new net LED_LOAD_BETWEEN_RESISTORS: R14.2, R26.1
- new net LED_LOAD_CATHODE: D1.2 (A), R26.2
- new net V_LOAD_FUSED: R14.1

Commit message: Finalize DC dimmer v0.1
Parts:
- D1: value LED -> LED_LOAD
- Q1: value Q_NMOS_GDS -> NCE0140KA
Changed lines of the file:
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@@
 			)
 		)
-		(property "Value" "Q_NMOS_GDS"
+		(property "Value" "NCE0140KA"
 			(at 138.43 96.5199 0)
 			(effects
@@
 			)
 		)
-		(property "Value" "LED"
+		(property "Value" "LED_LOAD"
 			(at 138.43 76.5174 90)
 			(effects

Commit message: Begin with improving dc dimmer
Parts:
- added F14: Fuse, pwm-ac-dimmer:fuseholder, symbol Device:Fuse
- added R46: 100R, Resistor_SMD:R_1206_3216Metric, symbol Device:R
- R3: value 300R -> 100R
- renumbered D1 to D, R14 to R
Connections:
- net GATE_SINK: no longer names the net of Q1.1 (G), R3.2
- net V_GATE: no longer names the net of R3.1
- net V_GATE: now also R46.2
- net V_LOAD_FUSED renamed LOAD_CATHODE
- net LOAD_CATHODE: now also F14.2
- new net GATE_DRIVE: R46.1
- new net V_LOAD: F14.1
Other:
- note added: "15 W light bulb = 0.3 A => 1A fuse"
- note added: "5V / 200R = 25 mA 2x 0805 resistors"
- note removed: "5V / 300R = 16 mA"
- moved on the sheet: R3
