File: pwm-dc-dimmer/pwm-dc-dimmer.kicad_sch (KiCad schematic)
At the start: 20 parts, among them J1 Screw_Terminal_01x02, J10 Screw_Terminal_01x02, J11 Screw_Terminal_01x02, J12 Screw_Terminal_01x02, J13 Screw_Terminal_01x02, J14 Conn_01x06_Pin, J16 Conn_01x06_Pin, J2 Screw_Terminal_01x02, J3 Screw_Terminal_01x02, J4 Screw_Terminal_01x02, J5 Screw_Terminal_01x02, J6 Screw_Terminal_01x02, J7 Screw_Terminal_01x02, J8 Screw_Terminal_01x02, J9 Screw_Terminal_01x02

Commit message: Add power routing
Parts:
- removed J14, J16: Conn_01x06_Pin, symbol Connector:Conn_01x06_Pin
- added C3: 100nF, Capacitor_SMD:C_0805_2012Metric, symbol Device:C_Small
- added C4: 10uF, Capacitor_SMD:C_1206_3216Metric, symbol Device:C_Small
- added D13: LED, LED_SMD:LED_0805_2012Metric, symbol Device:LED
- added F1: Fuse, pwm-ac-dimmer:fuseholder, symbol Device:Fuse
- added H1, H2, H3, H4: MountingHole, MountingHole:MountingHole_2.7mm_M2.5_ISO7380, symbol Mechanical:MountingHole
- added J14, J15: Conn_02x03_Odd_Even, Connector_IDC:IDC-Header_2x03_P2.54mm_Vertical, symbol Connector_Generic:Conn_02x03_Odd_Even
- added R38, R39: 10K, Resistor_SMD:R_0805_2012Metric, symbol Device:R
- C1: footprint (none) -> Capacitor_SMD:C_0805_2012Metric
- C2: footprint (none) -> Capacitor_SMD:C_1206_3216Metric
- J1, J10, J11, J12, J13, J2, J3, J4, J5, J6, J7, J8, J9: footprint (none) -> TerminalBlock_Phoenix:TerminalBlock_Phoenix_MKDS-1,5-2-5.08_1x02_P5.08mm_Horizontal
- NT1: footprint (none) -> NetTie:NetTie-2_THT_Pad1.0mm
- R1: footprint (none) -> Resistor_SMD:R_0805_2012Metric
- U1: footprint (none) -> Package_SO:HTSSOP-20-1EP_4.4x6.5mm_P0.65mm_EP3.4x6.5mm_ThermalVias
Connections:
- net GND: now also U1.21 (EP), C3.2, C4.2, J14.3 (Pin_3), J14.5 (Pin_5), J15.3 (Pin_3), J15.5 (Pin_5)
- net SCKI: now also J15.4 (Pin_4)
- net SCKO: now also J14.4 (Pin_4)
- net SDTI: now also J15.6 (Pin_6)
- net SDTO: now also J14.6 (Pin_6)
- net V_GATE: now also C3.1, C4.1, J14.1 (Pin_1), J15.1 (Pin_1)
- net V_LOAD: now also F1.1, R38.1; no longer J1.1 (Pin_1), J10.1 (Pin_1), J11.1 (Pin_1), J12.1 (Pin_1), J2.1 (Pin_1), J3.1 (Pin_1), J4.1 (Pin_1), J5.1 (Pin_1), J6.1 (Pin_1), J7.1 (Pin_1), J8.1 (Pin_1), J9.1 (Pin_1)
- net V_LOGIC: now also J14.2 (Pin_2), J15.2 (Pin_2)
- new net FUSE_LED_CATHODE: D13.2 (A), R39.2
- new net FUSE_LED_RESISTORS: R38.2, R39.1
- new net V_LOAD_FUSED: D13.1 (K), F1.2, J1.1 (Pin_1), J10.1 (Pin_1), J11.1 (Pin_1), J12.1 (Pin_1), J2.1 (Pin_1), J3.1 (Pin_1), J4.1 (Pin_1), J5.1 (Pin_1), J6.1 (Pin_1), J7.1 (Pin_1), J8.1 (Pin_1), J9.1 (Pin_1)
Other:
- note added: "Dimmer Channels"
- note added: "INPUT"
- note added: "Inputs"
- note added: "Mounting Holes"
- note added: "OUTPUT"
- note added: "Outputs"
- note added: "Power"
- note added: "~10A"
- moved on the sheet: C1, C2, J1, J10, J11, J12, J13, J2, J3, J4, J5, J6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

Commit message: Finalize DC dimmer v0.1
Parts:
- D13: value LED -> LED_FUSE
Changed lines of the file:
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@@
 			)
 		)
-		(property "Value" "LED"
+		(property "Value" "LED_FUSE"
 			(at 67.31 106.9974 90)
 			(effects

Commit message: Begin with improving dc dimmer
Parts:
- added C5, C7: 100nF, Capacitor_SMD:C_0805_2012Metric, symbol Device:C_Small
- added C6, C8: 10uF, Capacitor_SMD:C_1206_3216Metric, symbol Device:C_Small
- added R14, R41, R42, R43, R44, R45, R58, R59, R60, R61: 300R, Resistor_SMD:R_1206_3216Metric, symbol Device:R
- added R40, R62: 1k, Resistor_SMD:R_1206_3216Metric, symbol Device:R
- added U2, U3: 74LS240, symbol 74xx:74LS240
- D13: value LED_FUSE -> LED_POWER
Connections:
- net GND: now also C5.2, C6.2, C7.2, C8.2, U2.1 (OEa), U2.10 (GND), U2.19 (OEb), U3.1 (OEa), U3.10 (GND), U3.19 (OEb)
- net GND_LOAD: now also D13.1 (K)
- net V_GATE: no longer C3.1, C4.1, J14.1 (Pin_1), J15.1 (Pin_1)
- net V_LOAD: no longer R38.1
- net V_LOAD_FUSED: now also R38.1; no longer D13.1 (K), J1.1 (Pin_1), J10.1 (Pin_1), J11.1 (Pin_1), J12.1 (Pin_1), J2.1 (Pin_1), J3.1 (Pin_1), J4.1 (Pin_1), J5.1 (Pin_1), J6.1 (Pin_1), J7.1 (Pin_1), J8.1 (Pin_1), J9.1 (Pin_1)
- net GATE_SINK_1 renamed PWM_SINK_1
- net PWM_SINK_1: now also R40.2, U2.2 (I0a)
- net GATE_SINK_10 renamed PWM_SINK_10
- net PWM_SINK_10: now also R59.2, U3.11 (I0b)
- net GATE_SINK_11 renamed PWM_SINK_11
- net PWM_SINK_11: now also R58.2, U3.13 (I1b)
- net GATE_SINK_12 renamed PWM_SINK_12
- net PWM_SINK_12: now also R14.2, U3.15 (I2b)
- net GATE_SINK_2 renamed PWM_SINK_2
- net PWM_SINK_2: now also R41.2, U2.4 (I1a)
- net GATE_SINK_3 renamed PWM_SINK_3
- net PWM_SINK_3: now also R42.2, U2.6 (I2a)
- net GATE_SINK_4 renamed PWM_SINK_4
- net PWM_SINK_4: now also R43.2, U2.11 (I0b)
- net GATE_SINK_5 renamed PWM_SINK_5
- net PWM_SINK_5: now also R44.2, U2.13 (I1b)
- net GATE_SINK_6 renamed PWM_SINK_6
- net PWM_SINK_6: now also R45.2, U2.15 (I2b)
- net GATE_SINK_7 renamed PWM_SINK_7
- net PWM_SINK_7: now also R62.2, U3.2 (I0a)
- net GATE_SINK_8 renamed PWM_SINK_8
- net PWM_SINK_8: now also R61.2, U3.4 (I1a)
- net GATE_SINK_9 renamed PWM_SINK_9
- net PWM_SINK_9: now also R60.2, U3.6 (I2a)
- new net +5V: C3.1, C4.1, C5.1, C6.1, C7.1, C8.1, J14.1 (Pin_1), J15.1 (Pin_1), R14.1, R40.1, R41.1, R42.1, R43.1, R44.1, R45.1, R58.1, R59.1, R60.1, R61.1, R62.1, U2.20 (VCC), U3.20 (VCC)
- new net GATE_DRIVE_1: U2.18 (O0a)
- new net GATE_DRIVE_10: U3.9 (O0b)
- new net GATE_DRIVE_11: U3.7 (O1b)
- new net GATE_DRIVE_12: U3.5 (O2b)
- new net GATE_DRIVE_2: U2.16 (O1a)
- new net GATE_DRIVE_3: U2.14 (O2a)
- new net GATE_DRIVE_4: U2.9 (O0b)
- new net GATE_DRIVE_5: U2.7 (O1b)
- new net GATE_DRIVE_6: U2.5 (O2b)
- new net GATE_DRIVE_7: U3.18 (O0a)
- new net GATE_DRIVE_8: U3.16 (O1a)
- new net GATE_DRIVE_9: U3.14 (O2a)
- new net OUT1+: J1.1 (Pin_1)
- new net OUT10+: J10.1 (Pin_1)
- new net OUT11+: J11.1 (Pin_1)
- new net OUT12+: J12.1 (Pin_1)
- new net OUT2+: J2.1 (Pin_1)
- new net OUT3+: J3.1 (Pin_1)
- new net OUT4+: J4.1 (Pin_1)
- new net OUT5+: J5.1 (Pin_1)
- new net OUT6+: J6.1 (Pin_1)
- new net OUT7+: J7.1 (Pin_1)
- new net OUT8+: J8.1 (Pin_1)
- new net OUT9+: J9.1 (Pin_1)
- no-connect marks 0 -> 8
Other:
- sheet Channel 1 ports: added GATE_DRIVE, LOAD_CATHODE, V_LOAD; removed GATE_SINK
- sheet Channel 10 ports: added GATE_DRIVE, LOAD_CATHODE, V_LOAD; removed GATE_SINK
- sheet Channel 11 ports: added GATE_DRIVE, LOAD_CATHODE, V_LOAD; removed GATE_SINK
- sheet Channel 12 ports: added GATE_DRIVE, LOAD_CATHODE, V_LOAD; removed GATE_SINK
- sheet Channel 2 ports: added GATE_DRIVE, LOAD_CATHODE, V_LOAD; removed GATE_SINK
- sheet Channel 3 ports: added GATE_DRIVE, LOAD_CATHODE, V_LOAD; removed GATE_SINK
- sheet Channel 4 ports: added GATE_DRIVE, LOAD_CATHODE, V_LOAD; removed GATE_SINK
- sheet Channel 5 ports: added GATE_DRIVE, LOAD_CATHODE, V_LOAD; removed GATE_SINK
- sheet Channel 6 ports: added GATE_DRIVE, LOAD_CATHODE, V_LOAD; removed GATE_SINK
- sheet Channel 7 ports: added GATE_DRIVE, LOAD_CATHODE, V_LOAD; removed GATE_SINK
- sheet Channel 8 ports: added GATE_DRIVE, LOAD_CATHODE, V_LOAD; removed GATE_SINK
- sheet Channel 9 ports: added GATE_DRIVE, LOAD_CATHODE, V_LOAD; removed GATE_SINK
- note added: "NOTE: This IC inverts the signal, such that the gate drive is low by default"
- note added: "Since the PWM outputs can only sink current, we pull up the signal to 5V 5V / 1k = 5 mA"
- moved on the sheet: C1, C2, D13, F1, J1, J10, J11, J12, J14, J2, J3, J4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
